File: PCB/DRV8353S_dev_board/DRV8353S_dev_board.sch (KiCad schematic (older format))
At the start: 139 parts, among them J1 HC_POWER, J2 MOT_LC, J3 SWD, J4 EXT_CMD, J5 PHASE, Q1 BSS84, Q2 CSD19502, Q3 CSD19502, Q4 CSD19502, Q5 CSD19502, Q6 CSD19502, Q7 CSD19502, SW1 B3U, SW2 B3U, SW3 B3U, SW4 B3U, SW5 DIP, U1 ECS-33B, U2 STM32F042K4Ux, U3 MIC5283-3.3ML-TR, U4 MIC5283-5.0ML-TR, U5 DRV8353SM

Commit message: Fixed silkscreen and added BOM
Other:
- note added: "- Voltage: 25V - 50V\n- Max Current: 100A\n- Cont. Current: 50A\n- Sensored 120 deg trap. commutation \n- For use with Flipsky 6384"
- note removed: "- Voltage: 25V - 50V\n- Max Current: 100A\n- Max Power: 4000W\n- Sensored 120 deg trap. commutation \n- For use with Flipsky 6384"
Changed lines of the file:
@@
 DRV8353SM Dev. Board
 Text Notes 4200 1300 0    50   Italic 0
-- Voltage: 25V - 50V\n- Max Current: 100A\n- Max Power: 4000W\n- Sensored 120 deg trap. commutation \n- For use with Flipsky 6384
+- Voltage: 25V - 50V\n- Max Current: 100A\n- Cont. Current: 50A\n- Sensored 120 deg trap. commutation \n- For use with Flipsky 6384
 Text Notes 5900 1150 0    50   Italic 0
 Evaluation prototype for\nopen source e-mobility\nplatform.

Commit message: Changed MCU due to low digikey stock. Also new routing
Parts:
- removed U2: STM32F042K4Ux, Package_DFN_QFN:QFN-32-1EP_5x5mm_P0.5mm_EP3.45x3.45mm, symbol DRV8353S_dev_board-rescue:STM32F042K4Ux-MCU_ST_STM32F0
- added C?: 1uF, Capacitor_SMD:C_0805_2012Metric, symbol DRV8353S_dev_board-rescue:C_Small-Device
- added R?: 2.2k, Resistor_SMD:R_0603_1608Metric, symbol DRV8353S_dev_board-rescue:R_Small-Device
- added U2: STM32F103TBUx, Package_DFN_QFN:QFN-36-1EP_6x6mm_P0.5mm_EP4.1x4.1mm, symbol MCU_ST_STM32F1:STM32F103TBUx
- J5: Digikey (none) -> WM11180-ND; Mouser WM11180-ND -> (none)
- R38, R39, R55: Digikey 541-3124-1-ND -> YAG5784CT-ND‎
Connections:
- wire segments 378 -> 395
- no-connect marks 4 -> 2
Other:
- moved on the sheet: C14, C15, C16
